Commit message: Simulation branch (work in progress... basically a 'git stash'): Adding some inertia parameters to the xacro file. launch files updated to not start control node.

File: allegro_hand_description/allegro_hand_description_left.xacro (robot description, xacro)
@@ -45,4 +45,10 @@
     <xacro:property name="limit_3_t_low" value="-0.262"/>
     <!-- ============================================================================= -->
+    <!-- Used for fixing robot to Gazebo 'base_link' -->
+    <link name="world"/>
+    <joint name="fixed" type="fixed">
+      <parent link="world"/>
+      <child link="base_link"/>
+    </joint>
     <!-- BASE -->
     <link name="base_link">
@@ -62,4 +68,12 @@
             </geometry>
         </collision>
+        <inertial>
+          <origin xyz="0 0 ${base_link_z/2}" rpy="0 0 0"/>
+          <mass value="1"/>
+          <inertia
+	      ixx="1.0" ixy="0.0" ixz="0.0"
+	      iyy="1.0" iyz="0.0"
+	      izz="1.0"/>
+        </inertial>
     </link>
     <!-- ============================================================================= -->

Commit message: Fixing more naming of links.

File: allegro_hand_description/allegro_hand_description_left.xacro (robot description, xacro)
@@ -46,5 +46,5 @@
     <!-- ============================================================================= -->
     <!-- BASE -->
-    <link name="base_link">
+    <link name="palm_link">
         <visual>
             <geometry>
@@ -126,5 +126,5 @@
                    lower="${limit_0_t_low-joint_safety_margin}"
                    upper="${limit_0_t_up-joint_safety_margin}"/>
-            <parent link="base_link"/>
+            <parent link="palm_link"/>
             <child link="link_${finger_num*4+0}"/>
             <origin rpy="${finger_angle_r} ${finger_angle_p} ${finger_angle_y}"
@@ -254,5 +254,5 @@
                    lower="${limit_0_low+joint_safety_margin}"
                    upper="${limit_0_up-joint_safety_margin}"/>
-            <parent link="base_link"/>
+            <parent link="palm_link"/>
             <child link="link_${finger_num*4+0}"/>
             <origin rpy="${finger_angle_r} 0 0"

File: allegro_hand_description/allegro_hand_description_right.xacro (robot description, xacro)
@@ -46,5 +46,5 @@
     <!-- ============================================================================= -->
     <!-- BASE -->
-    <link name="base_link">
+    <link name="palm_link">
         <visual>
             <geometry>
@@ -124,5 +124,5 @@
                    lower="${limit_0_t_low-joint_safety_margin}"
                    upper="${limit_0_t_up-joint_safety_margin}"/>
-            <parent link="base_link"/>
+            <parent link="palm_link"/>
             <child link="link_${finger_num*4+0}"/>
             <origin rpy="${finger_angle_r} ${finger_angle_p} ${finger_angle_y}"
@@ -252,5 +252,5 @@
                    lower="${limit_0_low+joint_safety_margin}"
                    upper="${limit_0_up-joint_safety_margin}"/>
-            <parent link="base_link"/>
+            <parent link="palm_link"/>
             <child link="link_${finger_num*4+0}"/>
             <origin rpy="${finger_angle_r} 0 0"
