Commit message: Added inertial parameters for all links on the hand.

File: allegro_hand_description/allegro_hand_description_right.urdf (robot description, URDF)
Before this commit: robot allegro_hand_right, 21 links, 20 joints
Links:
- link link_0.0: mass None -> 0.0119
- link link_1.0: mass None -> 0.065
- link link_10.0: mass None -> 35.5
- link link_11.0: mass None -> 0.0096
- link link_11.0_tip: mass None -> 0.0168
- link link_12.0: mass None -> 0.176
- link link_13.0: mass None -> 0.0119
- link link_14.0: mass None -> 0.038
- link link_15.0: mass None -> 0.388
- link link_15.0_tip: mass None -> 0.0168
- link link_2.0: mass None -> 35.5
- link link_3.0: mass None -> 0.0096
- link link_3.0_tip: mass None -> 0.0168
- link link_4.0: mass None -> 0.0119
- link link_5.0: mass None -> 0.065
- link link_6.0: mass None -> 35.5
- link link_7.0: mass None -> 0.0096
- link link_7.0_tip: mass None -> 0.0168
- link link_8.0: mass None -> 0.0119
- link link_9.0: mass None -> 0.065

Commit message: Fixing inertial stuff.

File: allegro_hand_description/allegro_hand_description_right.urdf (robot description, URDF)
Before this commit: robot allegro_hand_right, 21 links, 20 joints
Links:
- link link_10.0: mass 35.5 -> 0.0355
- link link_12.0: mass 0.176 -> 0.0176
- link link_15.0: mass 0.388 -> 0.0388
- link link_2.0: mass 35.5 -> 0.0355
- link link_6.0: mass 35.5 -> 0.0355
Joints:
- joint joint_0.0: limit lower=-0.47 upper=0.47 effort=0 velocity=0 -> lower=-0.47 upper=0.47 effort=15 velocity=7
- joint joint_1.0: limit lower=-0.196 upper=1.61 effort=0 velocity=0 -> lower=-0.196 upper=1.61 effort=15 velocity=7
- joint joint_10.0: limit lower=-0.174 upper=1.709 effort=0 velocity=0 -> lower=-0.174 upper=1.709 effort=15 velocity=7
- joint joint_11.0: limit lower=-0.227 upper=1.618 effort=0 velocity=0 -> lower=-0.227 upper=1.618 effort=15 velocity=7
- joint joint_11.0_tip: limit (none) -> lower=0 upper=0 effort=.1 velocity=.1
- joint joint_12.0: limit lower=0.263 upper=1.396 effort=0 velocity=0 -> lower=0.263 upper=1.396 effort=15 velocity=7
- joint joint_13.0: limit lower=-0.105 upper=1.163 effort=0 velocity=0 -> lower=-0.105 upper=1.163 effort=15 velocity=7
- joint joint_14.0: limit lower=-0.189 upper=1.644 effort=0 velocity=0 -> lower=-0.189 upper=1.644 effort=15 velocity=7
- joint joint_15.0: limit lower=-0.162 upper=1.719 effort=0 velocity=0 -> lower=-0.162 upper=1.719 effort=15 velocity=7
- joint joint_15.0_tip: limit (none) -> lower=0 upper=0 effort=.1 velocity=.1
- joint joint_2.0: limit lower=-0.174 upper=1.709 effort=0 velocity=0 -> lower=-0.174 upper=1.709 effort=15 velocity=7
- joint joint_3.0: limit lower=-0.227 upper=1.618 effort=0 velocity=0 -> lower=-0.227 upper=1.618 effort=15 velocity=7
- joint joint_3.0_tip: limit (none) -> lower=0 upper=0 effort=.1 velocity=.1
- joint joint_4.0: limit lower=-0.47 upper=0.47 effort=0 velocity=0 -> lower=-0.47 upper=0.47 effort=15 velocity=7
- joint joint_5.0: limit lower=-0.196 upper=1.61 effort=0 velocity=0 -> lower=-0.196 upper=1.61 effort=15 velocity=7
- joint joint_6.0: limit lower=-0.174 upper=1.709 effort=0 velocity=0 -> lower=-0.174 upper=1.709 effort=15 velocity=7
- joint joint_7.0: limit lower=-0.227 upper=1.618 effort=0 velocity=0 -> lower=-0.227 upper=1.618 effort=15 velocity=7
- joint joint_7.0_tip: limit (none) -> lower=0 upper=0 effort=.1 velocity=.1
- joint joint_8.0: limit lower=-0.47 upper=0.47 effort=0 velocity=0 -> lower=-0.47 upper=0.47 effort=15 velocity=7
- joint joint_9.0: limit lower=-0.196 upper=1.61 effort=0 velocity=0 -> lower=-0.196 upper=1.61 effort=15 velocity=7

Commit message: Set friction and damping constants to make the hand not explode.

File: allegro_hand_description/allegro_hand_description_right.urdf (robot description, URDF)
Before this commit: robot allegro_hand_right, 21 links, 20 joints
Joints:
- joint joint_11.0_tip: limit lower=0 upper=0 effort=.1 velocity=.1 -> (none)
- joint joint_15.0_tip: limit lower=0 upper=0 effort=.1 velocity=.1 -> (none)
- joint joint_3.0_tip: limit lower=0 upper=0 effort=.1 velocity=.1 -> (none)
- joint joint_7.0_tip: limit lower=0 upper=0 effort=.1 velocity=.1 -> (none)

Commit message: Renamed 'base_link' to 'palm_link' to be more specific when adding hand to other robots. Changed defaults on launch file to make my life easier.

File: allegro_hand_description/allegro_hand_description_right.urdf (robot description, URDF)
Before this commit: robot allegro_hand_right, 21 links, 20 joints
Links:
- removed link base_link
- added link palm_link; collision box size=0.0408 0.1130 0.095; visual mesh filename=package://allegro_hand_description/meshes/base_link.STL
Joints:
- joint joint_0.0: parent base_link -> palm_link
- joint joint_12.0: parent base_link -> palm_link
- joint joint_4.0: parent base_link -> palm_link
- joint joint_8.0: parent base_link -> palm_link

Commit message: Changing frame names in URDF.
Need to make xacro match.

File: allegro_hand_description/allegro_hand_description_right.urdf (robot description, URDF)
Before this commit: robot allegro_hand_right, 21 links, 20 joints
Links:
- removed link link_11.0_tip
- removed link link_15.0_tip
- removed link link_3.0_tip
- removed link link_7.0_tip
- added link index_tip, mass 0.0168; collision sphere radius=0.012; visual mesh filename=package://allegro_hand_description/meshes/link_3.0_tip.STL
- added link middle_tip, mass 0.0168; collision sphere radius=0.012; visual mesh filename=package://allegro_hand_description/meshes/link_3.0_tip.STL
- added link ring_tip, mass 0.0168; collision sphere radius=0.012; visual mesh filename=package://allegro_hand_description/meshes/link_3.0_tip.STL
- added link thumb_tip, mass 0.0168; collision sphere radius=0.012; visual mesh filename=package://allegro_hand_description/meshes/link_15.0_tip.STL
Joints:
- joint joint_11.0_tip: child link_11.0_tip -> ring_tip
- joint joint_15.0_tip: child link_15.0_tip -> thumb_tip
- joint joint_3.0_tip: child link_3.0_tip -> index_tip
- joint joint_7.0_tip: child link_7.0_tip -> middle_tip

Commit message: Fixed robot description naming for thumb. Will do the same for the other fingers.

File: allegro_hand_description/allegro_hand_description_right.urdf (robot description, URDF)
Before this commit: robot allegro_hand_right, 21 links, 20 joints
Links:
- removed link link_12.0
- removed link link_13.0
- removed link link_14.0
- removed link link_15.0
- added link thumb_link_0, mass 0.0176; collision box size=0.0358 0.034 0.0455; visual mesh filename=package://allegro_hand_description/meshes/link_12.0_right.S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
- added link thumb_link_1, mass 0.0119; collision box size=0.0196 0.0275 0.0177; visual mesh filename=package://allegro_hand_description/meshes/link_13.0.STL
- added link thumb_link_2, mass 0.038; collision box size=0.0196 0.0275 0.0514; visual mesh filename=package://allegro_hand_description/meshes/link_14.0.STL
- added link thumb_link_3, mass 0.0388; collision box size=0.0196 0.0275 0.0423; visual mesh filename=package://allegro_hand_description/meshes/link_15.0.STL
Joints:
- removed joint joint_12.0
- removed joint joint_13.0
- removed joint joint_14.0
- removed joint joint_15.0
- removed joint joint_15.0_tip
- added joint thumb_joint_0: type revolute, parent palm_link, child thumb_link_0, origin xyz=-0.0182 0.019333 -0.045987 rpy=0 -1.65806278845 -1.5707963259, axis -1 0 0, limit lower=0.263 upper=1.396 effort=15 velocity=7
- added joint thumb_joint_1: type revolute, parent thumb_link_0, child thumb_link_1, origin xyz=-0.027 0.005 0.0399, axis 0 0 1, limit lower=-0.105 upper=1.163 effort=15 velocity=7
- added joint thumb_joint_2: type revolute, parent thumb_link_1, child thumb_link_2, origin xyz=0 0 0.0177, axis 0 1 0, limit lower=-0.189 upper=1.644 effort=15 velocity=7
- added joint thumb_joint_3: type revolute, parent thumb_link_2, child thumb_link_3, origin xyz=0 0 0.0514, axis 0 1 0, limit lower=-0.162 upper=1.719 effort=15 velocity=7
- added joint thumb_tip_joint: type fixed, parent thumb_link_3, child thumb_tip, origin xyz=0 0 0.0423 rpy=0 0 0

File: allegro_hand_description/allegro_hand_description_right.xacro (robot description, xacro)
@@ -68,4 +68,5 @@
     <!-- for LEFT HAND switch the sign of the **offset_origin_y** and **finger_angle_r** parameters-->
     <xacro:finger
+	    finger_name="index"
             finger_num="0"
             offset_origin_x="${offset_origin_x_const}"
@@ -75,4 +76,5 @@
             />
     <xacro:finger
+	    finger_name="middle"
             finger_num="1"
             offset_origin_x="${offset_origin_x_const}"
@@ -82,4 +84,5 @@
             />
     <xacro:finger
+	    finger_name="ring"
             finger_num="2"
             offset_origin_x="${offset_origin_x_const}"
@@ -90,4 +93,5 @@
     <!-- THUMB -->
     <xacro:thumb_right
+	    finger_name="thumb"
             finger_num="3"
             offset_origin_x="-0.0182"
@@ -101,7 +105,7 @@
     <!-- THUMB MACRO -->
     <xacro:macro name="thumb_right"
-                 params="finger_num offset_origin_x offset_origin_y offset_origin_z finger_angle_r finger_angle_p finger_angle_y">
+                 params="finger_name finger_num offset_origin_x offset_origin_y offset_origin_z finger_angle_r finger_angle_p finger_angle_y">
         <!-- [LINK 12] -->
-        <link name="link_${finger_num*4+0}">
+        <link name="${finger_name}_link_0">
             <visual>
                 <geometry>
@@ -119,5 +123,5 @@
             </collision>
         </link>
-        <joint name="joint_${finger_num*4+0}" type="revolute">
+        <joint name="${finger_name}_joint_0" type="revolute">
             <axis xyz="-1 0 0"/>
             <limit effort="0" velocity="0"
@@ -125,10 +129,10 @@
                    upper="${limit_0_t_up-joint_safety_margin}"/>
             <parent link="palm_link"/>
-            <child link="link_${finger_num*4+0}"/>
+            <child link="${finger_name}_link_0"/>
             <origin rpy="${finger_angle_r} ${finger_angle_p} ${finger_angle_y}"
                     xyz="${offset_origin_x} ${offset_origin_y} ${offset_origin_z}"/>
         </joint>
         <!-- [LINK 13] -->
-        <link name="link_${finger_num*4+1}">
+        <link name="${finger_name}_link_1">
             <visual>
                 <geometry>
@@ -146,15 +150,15 @@
             </collision>
         </link>
-        <joint name="joint_${finger_num*4+1}" type="revolute">
+        <joint name="${finger_name}_joint_1" type="revolute">
             <axis xyz="0 0 1"/>
             <limit effort="0" velocity="0"
                    lower="${limit_1_t_low+joint_safety_margin}"
                    upper="${limit_1_t_up-joint_safety_margin}"/>
-            <parent link="link_${finger_num*4+0}"/>
-            <child link="link_${finger_num*4+1}"/>
+            <parent link="${finger_name}_link_0"/>
+            <child link="${finger_name}_link_1"/>
             <origin xyz="-0.027 0.005 0.0399"/>
         </joint>
         <!-- [LINK 14] -->
-        <link name="link_${finger_num*4+2}">
+        <link name="${finger_name}_link_2">
             <visual>
                 <geometry>
@@ -171,15 +175,15 @@
             </collision>
         </link>
-        <joint name="joint_${finger_num*4+2}" type="revolute">
+        <joint name="${finger_name}_joint_2" type="revolute">
             <axis xyz="0 1 0"/>
             <limit effort="0" velocity="0"
                    lower="${limit_2_t_low+joint_safety_margin}"
                    upper="${limit_2_t_up-joint_safety_margin}"/>
-            <parent link="link_${finger_num*4+1}"/>
-            <child link="link_${finger_num*4+2}"/>
+            <parent link="${finger_name}_link_1"/>
+            <child link="${finger_name}_link_2"/>
             <origin xyz="0 0 ${link1_t_z}"/>
         </joint>
         <!-- [LINK 15] -->
-        <link name="link_${finger_num*4+3}">
+        <link name="${finger_name}_link_3">
             <visual>
                 <geometry>
@@ -196,15 +200,15 @@
             </collision>
         </link>
-        <joint name="joint_${finger_num*4+3}" type="revolute">
+        <joint name="${finger_name}_joint_3" type="revolute">
             <axis xyz="0 1 0"/>
             <limit effort="0" velocity="0"
                    lower="${limit_3_t_low+joint_safety_margin}"
                    upper="${limit_3_t_up-joint_safety_margin}"/>
-            <parent link="link_${finger_num*4+2}"/>
-            <child link="link_${finger_num*4+3}"/>
+            <parent link="${finger_name}_link_2"/>
+            <child link="${finger_name}_link_3"/>
             <origin xyz="0 0 ${link2_t_z}"/>
         </joint>
         <!-- [FINGER TIP] -->
-        <link name="link_${finger_num*4+3}_tip">
+        <link name="${finger_name}_tip">
             <visual>
                 <geometry>
@@ -222,7 +226,7 @@
             </collision>
         </link>
-        <joint name="joint_${finger_num*4+3}_tip" type="fixed">
-            <parent link="link_${finger_num*4+3}"/>
-            <child link="link_${finger_num*4+3}_tip"/>
+        <joint name="${finger_name}_tip_joint" type="fixed">
+            <parent link="${finger_name}_link_3"/>
+            <child link="${finger_name}_tip"/>
             <origin rpy="0 0 0" xyz="0 0 ${link3_t_z-fingerTip_r}"/>
         </joint>
@@ -231,5 +235,5 @@
     <!-- THREE FINGER MACRO -->
     <xacro:macro name="finger"
-                 params="finger_num offset_origin_x offset_origin_y offset_origin_z finger_angle_r">
+                 params="finger_name finger_num offset_origin_x offset_origin_y offset_origin_z finger_angle_r">
         <!-- [LINK 0, 4, 8] -->
         <link name="link_${finger_num*4+0}">

Commit message: Updating rest of the finger names to be easier to understand.

File: allegro_hand_description/allegro_hand_description_right.urdf (robot description, URDF)
Before this commit: robot allegro_hand_right, 21 links, 20 joints
Links:
- removed link link_0.0
- removed link link_1.0
- removed link link_10.0
- removed link link_11.0
- removed link link_2.0
- removed link link_3.0
- removed link link_4.0
- removed link link_5.0
- removed link link_6.0
- removed link link_7.0
- removed link link_8.0
- removed link link_9.0
- added link index_link_0, mass 0.0119; collision box size=0.0196 0.0275 0.0164; visual mesh filename=package://allegro_hand_description/meshes/link_0.0.STL
- added link index_link_1, mass 0.065; collision box size=0.0196 0.0275 0.054; visual mesh filename=package://allegro_hand_description/meshes/link_1.0.STL
- added link index_link_2, mass 0.0355; collision box size=0.0196 0.0275 0.0384; visual mesh filename=package://allegro_hand_description/meshes/link_2.0.STL
- added link index_link_3, mass 0.0096; collision box size=0.0196 0.0275 0.0267; visual mesh filename=package://allegro_hand_description/meshes/link_3.0.STL
- added link middle_link_0, mass 0.0119; collision box size=0.0196 0.0275 0.0164; visual mesh filename=package://allegro_hand_description/meshes/link_0.0.STL
- added link middle_link_1, mass 0.065; collision box size=0.0196 0.0275 0.054; visual mesh filename=package://allegro_hand_description/meshes/link_1.0.STL
- added link middle_link_2, mass 0.0355; collision box size=0.0196 0.0275 0.0384; visual mesh filename=package://allegro_hand_description/meshes/link_2.0.STL
- added link middle_link_3, mass 0.0096; collision box size=0.0196 0.0275 0.0267; visual mesh filename=package://allegro_hand_description/meshes/link_3.0.STL
- added link ring_link_0, mass 0.0119; collision box size=0.0196 0.0275 0.0164; visual mesh filename=package://allegro_hand_description/meshes/link_0.0.STL
- added link ring_link_1, mass 0.065; collision box size=0.0196 0.0275 0.054; visual mesh filename=package://allegro_hand_description/meshes/link_1.0.STL
- added link ring_link_2, mass 0.0355; collision box size=0.0196 0.0275 0.0384; visual mesh filename=package://allegro_hand_description/meshes/link_2.0.STL
- added link ring_link_3, mass 0.0096; collision box size=0.0196 0.0275 0.0267; visual mesh filename=package://allegro_hand_description/meshes/link_3.0.STL
Joints:
- removed joint joint_0.0
- removed joint joint_1.0
- removed joint joint_10.0
- removed joint joint_11.0
- removed joint joint_11.0_tip
- removed joint joint_2.0
- removed joint joint_3.0
- removed joint joint_3.0_tip
- removed joint joint_4.0
- removed joint joint_5.0
- removed joint joint_6.0
- removed joint joint_7.0
- removed joint joint_7.0_tip
- removed joint joint_8.0
- removed joint joint_9.0
- added joint index_joint_0: type revolute, parent palm_link, child index_link_0, origin xyz=0 0.0435 -0.001542 rpy=-0.08726646255 0 0, axis 0 0 1, limit lower=-0.47 upper=0.47 effort=15 velocity=7
- added joint index_joint_1: type revolute, parent index_link_0, child index_link_1, origin xyz=0 0 0.0164, axis 0 1 0, limit lower=-0.196 upper=1.61 effort=15 velocity=7
- added joint index_joint_2: type revolute, parent index_link_1, child index_link_2, origin xyz=0 0 0.054, axis 0 1 0, limit lower=-0.174 upper=1.709 effort=15 velocity=7
- added joint index_joint_3: type revolute, parent index_link_2, child index_link_3, origin xyz=0 0 0.0384, axis 0 1 0, limit lower=-0.227 upper=1.618 effort=15 velocity=7
- added joint index_tip_joint: type fixed, parent index_link_3, child index_tip, origin xyz=0 0 0.0267 rpy=0 0 0
- added joint middle_joint_0: type revolute, parent palm_link, child middle_link_0, origin xyz=0 0 0.0007 rpy=0.0 0 0, axis 0 0 1, limit lower=-0.47 upper=0.47 effort=15 velocity=7
- added joint middle_joint_1: type revolute, parent middle_link_0, child middle_link_1, origin xyz=0 0 0.0164, axis 0 1 0, limit lower=-0.196 upper=1.61 effort=15 velocity=7
- added joint middle_joint_2: type revolute, parent middle_link_1, child middle_link_2, origin xyz=0 0 0.054, axis 0 1 0, limit lower=-0.174 upper=1.709 effort=15 velocity=7
- added joint middle_joint_3: type revolute, parent middle_link_2, child middle_link_3, origin xyz=0 0 0.0384, axis 0 1 0, limit lower=-0.227 upper=1.618 effort=15 velocity=7
- added joint middle_tip_joint: type fixed, parent middle_link_3, child middle_tip, origin xyz=0 0 0.0267 rpy=0 0 0
- added joint ring_joint_0: type revolute, parent palm_link, child ring_link_0, origin xyz=0 -0.0435 -0.001542 rpy=0.08726646255 0 0, axis 0 0 1, limit lower=-0.47 upper=0.47 effort=15 velocity=7
- added joint ring_joint_1: type revolute, parent ring_link_0, child ring_link_1, origin xyz=0 0 0.0164, axis 0 1 0, limit lower=-0.196 upper=1.61 effort=15 velocity=7
- added joint ring_joint_2: type revolute, parent ring_link_1, child ring_link_2, origin xyz=0 0 0.054, axis 0 1 0, limit lower=-0.174 upper=1.709 effort=15 velocity=7
- added joint ring_joint_3: type revolute, parent ring_link_2, child ring_link_3, origin xyz=0 0 0.0384, axis 0 1 0, limit lower=-0.227 upper=1.618 effort=15 velocity=7
- added joint ring_tip_joint: type fixed, parent ring_link_3, child ring_tip, origin xyz=0 0 0.0267 rpy=0 0 0

File: allegro_hand_description/allegro_hand_description_right.xacro (robot description, xacro)
@@ -237,5 +237,5 @@
                  params="finger_name finger_num offset_origin_x offset_origin_y offset_origin_z finger_angle_r">
         <!-- [LINK 0, 4, 8] -->
-        <link name="link_${finger_num*4+0}">
+        <link name="${finger_name}_link_0">
             <visual>
                 <geometry>
@@ -257,10 +257,10 @@
                    upper="${limit_0_up-joint_safety_margin}"/>
             <parent link="palm_link"/>
-            <child link="link_${finger_num*4+0}"/>
+            <child link="${finger_name}_link_0"/>
             <origin rpy="${finger_angle_r} 0 0"
                     xyz="${offset_origin_x} ${offset_origin_y} ${offset_origin_z}"/>
         </joint>
         <!-- [LINK 1, 5, 9] -->
-        <link name="link_${finger_num*4+1}">
+        <link name="${finger_name}_link_1">
             <visual>
                 <geometry>
@@ -281,10 +281,10 @@
                    upper="${limit_1_up-joint_safety_margin}"/>
             <axis xyz="0 1 0"/>
-            <parent link="link_${finger_num*4+0}"/>
-            <child link="link_${finger_num*4+1}"/>
+            <parent link="${finger_name}_link_0"/>
+            <child link="${finger_name}_link_1"/>
             <origin xyz="0 0 ${link0_z}"/>
         </joint>
         <!-- [LINK 2, 6, 10]-->
-        <link name="link_${finger_num*4+2}">
+        <link name="${finger_name}_link_2">
             <visual>
                 <geometry>
@@ -305,10 +305,10 @@
                    lower="${limit_2_low+joint_safety_margin}"
                    upper="${limit_2_up-joint_safety_margin}"/>
-            <parent link="link_${finger_num*4+1}"/>
-            <child link="link_${finger_num*4+2}"/>
+            <parent link="${finger_name}_link_1"/>
+            <child link="${finger_name}_link_2"/>
             <origin xyz="0 0 ${link1_z}"/>
         </joint>
         <!-- [LINK 3, 7, 11] -->
-        <link name="link_${finger_num*4+3}">
+        <link name="${finger_name}_link_3">
             <visual>
                 <geometry>
@@ -329,10 +329,10 @@
                    lower="${limit_3_low+joint_safety_margin}"
                    upper="${limit_3_up-joint_safety_margin}"/>
-            <parent link="link_${finger_num*4+2}"/>
-            <child link="link_${finger_num*4+3}"/>
+            <parent link="${finger_name}_link_2"/>
+            <child link="${finger_name}_link_3"/>
             <origin xyz="0 0 ${link2_z}"/>
         </joint>
         <!-- [FINGER TIP] -->
-        <link name="link_${finger_num*4+3}_tip">
+        <link name="${finger_name}_tip">
             <visual>
                 <geometry>
@@ -350,6 +350,6 @@
         </link>
         <joint name="joint_${finger_num*4+3}_tip" type="fixed">
-            <parent link="link_${finger_num*4+3}"/>
-            <child link="link_${finger_num*4+3}_tip"/>
+            <parent link="${finger_name}_link_3"/>
+            <child link="${finger_name}_tip"/>
             <origin rpy="0 0 0" xyz="0 0 ${link3_z-fingerTip_r}"/>
         </joint>
